Commit message: improve the go home motion

File: cute_model/robots/cute_300es.urdf.xacro (robot description, xacro)
@@ -5,4 +5,6 @@
   <xacro:include filename="$(find cute_model)/robots/cute_transmission.xacro" />
   <xacro:property name="PI" value="3.1415926535897931"/>
+  <xacro:property name="horizontal_joint_limit" value="2.61799"/>
+  <xacro:property name="vertical_joint_limit" value="1.8326"/>
   <link name="world"/>
   <joint name="world_base" type="fixed">
@@ -100,6 +102,6 @@
       xyz="0 0 1" />
     <limit
-      lower="${-0.58*PI}"
-      upper="${0.58*PI}"
+      lower="${-1*horizontal_joint_limit}"
+      upper="${horizontal_joint_limit}"
       effort="120"
       velocity="4.0" />
@@ -154,6 +156,6 @@
       xyz="0 1 0" />
     <limit
-      lower="${-0.58*PI}"
-      upper="${0.58*PI}"
+      lower="${-1*vertical_joint_limit}"
+      upper="${vertical_joint_limit}"
       effort="120"
       velocity="4.0" />
@@ -208,6 +210,6 @@
       xyz="0 0 1" />
     <limit
-      lower="${-0.58*PI}"
-      upper="${0.58*PI}"
+      lower="${-1*horizontal_joint_limit}"
+      upper="${horizontal_joint_limit}"
       effort="120"
       velocity="4.0" />
@@ -262,6 +264,6 @@
       xyz="0 1 0" />
     <limit
-      lower="${-0.58*PI}"
-      upper="${0.58*PI}"
+      lower="${-1*vertical_joint_limit}"
+      upper="${vertical_joint_limit}"
       effort="120"
       velocity="4.0" />
@@ -316,6 +318,6 @@
       xyz="0 -1 0" />
     <limit
-      lower="${-0.58*PI}"
-      upper="${0.58*PI}"
+      lower="${-1*vertical_joint_limit}"
+      upper="${vertical_joint_limit}"
       effort="120"
       velocity="4.0" />
@@ -370,6 +372,6 @@
       xyz="-0.24105 0.97051 0" />
     <limit
-      lower="${-0.58*PI}"
-      upper="${0.58*PI}"
+      lower="${-1*vertical_joint_limit}"
+      upper="${vertical_joint_limit}"
       effort="120"
       velocity="4.0" />
@@ -424,6 +426,6 @@
       xyz="0 0 1" />
     <limit
-      lower="${-0.58*PI}"
-      upper="${0.58*PI}"
+      lower="${-1*horizontal_joint_limit}"
+      upper="${horizontal_joint_limit}"
       effort="120"
       velocity="4.0" />
